Commit message: Rename chassis to base_linnk to fit convention

File: simulation/marvin_simulation/urdf/camera.xacro (robot description, xacro)
@@ -28,5 +28,5 @@
         <joint name="sim_camera_joint" type="fixed">
             <xacro:insert_block name="joint_origin" />
-            <parent link="chassis" />
+            <parent link="base_link" />
             <child link="camera" />
             <axis xyz="0 1 0" />

File: simulation/marvin_simulation/urdf/marvin.xacro (robot description, xacro)
@@ -43,5 +43,5 @@
 	<xacro:include filename="$(find marvin_simulation)/urdf/inertia.xacro" />
 	<!-- Chassis -->
-	<link name="chassis">
+	<link name="base_link">
 		<visual name="chassis_tower_visual">
 			<origin xyz="0 0 ${chassis_tower_height / 2 + chassis_z_offset}" rpy="0 0 0" />
@@ -111,5 +111,5 @@
     <joint name="caster_joint" type="fixed">
         <origin xyz="${caster_x_offset} 0 ${caster_radius}" rpy="0 0 0" />
-        <parent link="chassis" />
+        <parent link="base_link" />
         <child link="caster" />
     </joint>
@@ -128,5 +128,5 @@
 	<joint name="zed_camera_joint" type="fixed">
 		<origin xyz="${camera_x_offset} 0 ${camera_z_offset + chassis_z_offset}" rpy="0 ${camera_angle} 0" />
-		<parent link="chassis" />
+		<parent link="base_link" />
 		<child link="zed_camera_link" />
 	</joint>
@@ -138,5 +138,5 @@
     <!-- Lidar -->
     <xacro:include filename="$(find velodyne_description)/urdf/VLP-16.urdf.xacro" />
-	<xacro:VLP-16 parent="chassis" name="velodyne" topic="/velodyne_points" hz="20" samples="440" gpu="true">
+	<xacro:VLP-16 parent="base_link" name="velodyne" topic="/velodyne_points" hz="20" samples="440" gpu="true">
 		<origin xyz="0 0 ${chassis_z_offset + lidar_height}" rpy="0 0 0" />
 	</xacro:VLP-16>
@@ -161,5 +161,5 @@
 	<joint name="imu_joint" type="fixed">
 		<origin xyz="${-chassis_tower_length / 2 - chassis_electrical_length/2+0.005} 0 ${chassis_electrical_height + chassis_z_offset}" rpy="0 0 0" />
-		<parent link="chassis" />
+		<parent link="base_link" />
 		<child link="imu_link" />
 		<axis xyz="0 1 0" />
@@ -169,5 +169,5 @@
 	<joint name="encoders_joint" type="fixed">
 		<origin xyz="0 0 ${wheel_radius}" rpy="0 0 0" />
-		<parent link="chassis" />
+		<parent link="base_link" />
 		<child link="encoders" />
 		<axis xyz="0 1 0" />

File: simulation/marvin_simulation/urdf/wheel.xacro (robot description, xacro)
@@ -22,5 +22,5 @@
         <joint type="continuous" name="${prefix}_wheel_joint">
             <xacro:insert_block name="joint_origin" />
-            <parent link="chassis" />
+            <parent link="base_link" />
             <child link="${prefix}_wheel" />
             <axis xyz="0 1 0" rpy="0 0 0" />
