Commit message: Rename marvin_new to marvin

File: simulation/marvin_simulation/urdf/marvin.xacro (robot description, xacro)
@@ -1,89 +1,131 @@
 <?xml version='1.0'?>
 <robot name="marvin" xmlns:xacro="http://www.ros.org/wiki/xacro">
-	<xacro:property name="front_offset" value="0.3" /> <!-- How far forward the wheels and lidar are compared to the center of the chassis -->
-	<xacro:property name="back_offset" value="-0.6715" /> <!-- How far back the caster wheel is compared to the center of the chassis -->
-	<xacro:property name="chassis_mass" value="29.9371" />
-	<xacro:property name="chassis_length" value="1.143" />
-	<xacro:property name="chassis_width" value="0.6096" />
-	<xacro:property name="chassis_height" value="0.5588" />
-	<!-- Center of mass (relative to center of chassis) -->
-	<xacro:property name="com_x" value="0.0" />
-	<xacro:property name="com_y" value="0.0" />
-	<xacro:property name="com_z" value="0.0" />
-	<xacro:property name="caster_radius" value="0.05" />
-	<xacro:property name="wheel_mass" value="5" />
-	<xacro:property name="wheel_radius" value="0.157226" />
-	<xacro:property name="wheel_width" value="0.15" />
-	<xacro:property name="wheel_separation" value="0.78" /> <!-- Distance from center to center -->
-	<xacro:property name="wheel_offset" value="0.01" /> <!-- How far above the bottom plate of the robot the wheels are -->
-	<xacro:property name="lidar_height" value="0.89535"/> <!-- The distance from the base of the chassis to the base of the LiDAR -->
-	<xacro:property name="camera_mass" value="0.1"/>
-	<xacro:property name="camera_front_offset" value="0.5715"/> <!-- How far forward the camera is compared to the center of the chassis -->
-	<xacro:property name="camera_z_offset" value="0.1"/> <!-- How far down the camera is compared to the LiDAR -->
+	<!-- Chassis Constants -->
+    <xacro:property name="chassis_length" value="${45.5*0.0254}" />
+    <xacro:property name="chassis_width" value="${24*0.0254}" />
+    <xacro:property name="chassis_height" value="${22*0.0254}" />
+    <xacro:property name="chassis_z_offset" value="${4.375*0.0254}" />
+    <xacro:property name="chassis_tower_length" value="${8*0.0254}" />
+    <xacro:property name="chassis_tower_height" value="${31*0.0254}" />
+    <xacro:property name="chassis_payload_length" value="${14.25*0.0254}" />
+    <xacro:property name="chassis_payload_height" value="${8*0.0254}" />
+    <xacro:property name="chassis_electrical_length" value="${15.25*0.0254}" />
+    <xacro:property name="chassis_electrical_height" value="${22*0.0254}" />
+    <xacro:property name="chassis_caster_length" value="${8*0.0254}" />
+    <xacro:property name="chassis_caster_height" value="${2.25*0.0254}" />
+    <xacro:property name="chassis_caster_z_offset" value="${2*0.0254}" />
+    <!-- Chassis Inertial Constants -->
+    <xacro:property name="chassis_mass" value="29.9371" />
+    <xacro:property name="com_x" value="0.0" />
+    <xacro:property name="com_y" value="0.0" />
+    <xacro:property name="com_z" value="${6.1875*0.0254}" />
+	<!-- Caster Constants -->
+    <xacro:property name="caster_x_offset" value="${-24.625*0.0254}" />
+    <xacro:property name="caster_radius" value="${3.5*0.0254}" />
+    <xacro:property name="caster_mass" value="0.1" />
+	<!-- Wheel Constants -->
+    <xacro:property name="wheel_radius" value="${6.1875*0.0254}" />
+    <xacro:property name="wheel_width" value="${4*0.0254}" />
+    <xacro:property name="wheel_mass" value="5" />
+    <xacro:property name="track_width" value="${31*0.0254}" />
+    <!-- Lidar Constants -->
+    <xacro:property name="lidar_height" value="${32.55*0.0254}"/>
+    <!-- Camera Constants -->
+    <xacro:property name="camera_mass" value="0.1"/>
+    <xacro:property name="camera_angle" value="${10 * 0.01745327777}"/>
+    <xacro:property name="camera_x_offset" value="${(4+2.66916)*0.0254}"/>
+    <xacro:property name="camera_z_offset" value="${(31-1.80395)*0.0254}"/>
+    <!-- IMU Constants -->
+    <xacro:property name="imu_mass" value="0.025"/>
+    <xacro:property name="imu_length" value="0.05"/>
+    <xacro:property name="imu_width" value="0.03"/>
+    <xacro:property name="imu_height" value="0.01"/>
+	<xacro:include filename="$(find marvin_simulation)/urdf/inertia.xacro" />
 	<!-- Chassis -->
 	<link name="chassis">
-		<origin xyz="0 0 0" rpy="0 0 0" />
-		<visual name="chassis_base_visual">
-			<origin xyz="0 0 0" rpy="0 0 0" />
-			<geometry>
-				<box size="${chassis_length} ${chassis_width} ${chassis_height}" />
+		<visual name="chassis_tower_visual">
+			<origin xyz="0 0 ${chassis_tower_height / 2 + chassis_z_offset}" rpy="0 0 0" />
+			<geometry>
+				<box size="${chassis_tower_length} ${chassis_width} ${chassis_tower_height}" />
 			</geometry>
 		</visual>
-		<visual name="chassis_top_visual">
-			<origin xyz="${chassis_length/2-chassis_length/6} 0 ${chassis_height-(lidar_height-chassis_height)/3}" rpy="0 0 0" />
-			<geometry>
-				<box size="${chassis_length/3} ${chassis_width} ${lidar_height-chassis_height}" />
-			</geometry>
-		</visual>
-		<visual name="chassis_front_visual">
-			<origin xyz="${chassis_length/2+0.15} 0 ${0.05-chassis_height/2}" rpy="0 0 0" />
-			<geometry>
-				<box size="0.3 ${chassis_width} 0.1" />
-			</geometry>
-		</visual>
-		<visual name="chassis_back_visual">
-			<origin xyz="${-chassis_length/2-0.1} 0 ${0.05-chassis_height/2}" rpy="0 0 0" />
-			<geometry>
-				<box size="0.2 ${chassis_width} 0.1" />
-			</geometry>
-		</visual>
-		<visual name='caster_visual'>
-			<origin xyz="${back_offset} 0 ${caster_radius+wheel_offset-wheel_radius-chassis_height/2}" rpy=" 0 0 0"/>
+        <visual name="chassis_payload_visual">
+            <origin xyz="${chassis_tower_length / 2 + chassis_payload_length / 2} 0 ${chassis_payload_height / 2 + chassis_z_offset}" rpy="0 0 0" />
+            <geometry>
+                <box size="${chassis_payload_length} ${chassis_width} ${chassis_payload_height}" />
+            </geometry>
+        </visual>
+        <visual name="chassis_electrical_visual">
+            <origin xyz="${-chassis_tower_length / 2 - chassis_electrical_length / 2} 0 ${chassis_electrical_height / 2 + chassis_z_offset}" rpy="0 0 0" />
+            <geometry>
+                <box size="${chassis_electrical_length} ${chassis_width} ${chassis_electrical_height}" />
+            </geometry>
+        </visual>
+        <visual name="chassis_caster_visual">
+            <origin xyz="${-chassis_tower_length / 2 - chassis_electrical_length - chassis_caster_length / 2}
+                         0
+                         ${chassis_caster_height / 2 + chassis_caster_z_offset + chassis_z_offset}"
+                         rpy="0 0 0" />
+            <geometry>
+                <box size="${chassis_caster_length} ${chassis_width} ${chassis_caster_height}" />
+            </geometry>
+        </visual>
+		<collision name="chassis_collision">
+			<origin xyz="${chassis_tower_length / 2 + chassis_payload_length - chassis_length / 2}
+                         0
+                         ${chassis_z_offset + chassis_tower_height / 2}"
+                    rpy="0 0 0" />
+			<geometry>
+				<box size="${chassis_length} ${chassis_width} ${chassis_tower_height}" />
+			</geometry>
+		</collision>
+        <xacro:box_inertia mass="${chassis_mass}" length="${chassis_length}" width="${chassis_width}" height="${chassis_height}">
+            <origin xyz="${com_x} ${com_y} ${com_z}" rpy="0 0 0" />
+		</xacro:box_inertia>
+	</link>
+    <!-- Caster -->
+    <link name="caster">
+        <visual name="caster_visual">
+            <geometry>
+                <sphere radius="${caster_radius}" />
+            </geometry>
+        </visual>
+        <collision name='caster_collision'>
+			<origin xyz="0 0 0" rpy=" 0 0 0"/>
 			<geometry>
 				<sphere radius="${caster_radius}"/>
 			</geometry>
-		</visual>
-	</link>
-	<!-- Chassis Inertia -->
-	<link name="chassis_inertial_link">
-		<inertial>
-			<mass value="${chassis_mass}" />
-			<origin xyz="${com_x} ${com_y} ${com_z}" rpy="0 0 0" />
-			<inertia
-				ixx="${chassis_mass/12*(chassis_height**2+chassis_length**2)}" ixy="0" ixz="0"
-				iyy="${chassis_mass/12*(chassis_width**2+chassis_height**2)}" iyz="0"
-				izz="${chassis_mass/12*(chassis_width**2+chassis_length**2)}"
-			/>
-		</inertial>
-	</link>
-	<joint name="chassis_inertial_joint" type="fixed">
-		<origin xyz="0 0 0" rpy="0 0 0" />
-		<parent link="chassis" />
-		<child link="chassis_inertial_link" />
-	</joint>
-	<!-- Wheels -->
-	<xacro:include filename="$(find marvin_simulation)/urdf/wheel.xacro"/>
+			<surface>
+				<friction>
+				<ode>
+					<mu>0.0</mu>
+					<mu2>0.0</mu2>
+				</ode>
+				</friction>
+			</surface>
+		</collision>
+        <xacro:sphere_inertia mass="${caster_mass}" radius="${caster_radius}">
+            <origin xyz="0 0 0" rpy="0 0 0" />
+        </xacro:sphere_inertia>
+    </link>
+    <joint name="caster_joint" type="fixed">
+        <origin xyz="${caster_x_offset} 0 ${caster_radius}" rpy="0 0 0" />
+        <parent link="chassis" />
+        <child link="caster" />
+    </joint>
+    <!-- Wheels -->
+    <xacro:include filename="$(find marvin_simulation)/urdf/wheel.xacro"/>
 	<xacro:wheel prefix="right" mass="${wheel_mass}" radius="${wheel_radius}" width="${wheel_width}">
-		<origin xyz="${front_offset} -${wheel_separation/2} ${wheel_offset-chassis_height/2}" rpy="0 0 0" />
+		<origin xyz="0 -${track_width / 2} ${wheel_radius}" rpy="0 0 0" />
 	</xacro:wheel>
 	<xacro:wheel prefix="left" mass="${wheel_mass}" radius="${wheel_radius}" width="${wheel_width}">
-		<origin xyz="${front_offset} ${wheel_separation/2} ${wheel_offset-chassis_height/2}" rpy="0 0 0" />
+		<origin xyz="0 ${track_width/2} ${wheel_radius}" rpy="0 0 0" />
 	</xacro:wheel>
-	<!-- ZED Camera -->
+    <!-- ZED Camera -->
 	<xacro:include filename="$(find zed_wrapper)/urdf/zed_macro.urdf.xacro" />
 	<xacro:zed_camera name="zed" model="zed">
 	</xacro:zed_camera>
 	<joint name="zed_camera_joint" type="fixed">
-		<origin xyz="${camera_front_offset} 0 ${lidar_height-chassis_height/2-camera_z_offset}" rpy="0 0 0" /> <!-- Rotation may be wrong -->
+		<origin xyz="${camera_x_offset} 0 ${camera_z_offset + chassis_z_offset}" rpy="0 ${camera_angle} 0" />
 		<parent link="chassis" />
 		<child link="zed_camera_link" />
@@ -92,10 +134,10 @@
 	<xacro:include filename="$(find marvin_simulation)/urdf/camera.xacro" />
 	<xacro:camera mass="${camera_mass}">
-		<origin xyz="${camera_front_offset} 0 ${lidar_height-chassis_height/2-camera_z_offset+0.03/2}" rpy="0 0 0" /> <!-- Rotation may be wrong -->
+		<origin xyz="${camera_x_offset} 0 ${camera_z_offset + chassis_z_offset}" rpy="0 ${camera_angle} 0" />
 	</xacro:camera>
-	<!-- LiDAR -->
-	<xacro:include filename="$(find velodyne_description)/urdf/VLP-16.urdf.xacro" />
+    <!-- Lidar -->
+    <xacro:include filename="$(find velodyne_description)/urdf/VLP-16.urdf.xacro" />
 	<xacro:VLP-16 parent="chassis" name="velodyne" topic="/velodyne_points" hz="20" samples="440" gpu="true">
-		<origin xyz="${chassis_length/2-chassis_length/6} 0 ${lidar_height-chassis_height/2}" rpy="0 0 0" />
+		<origin xyz="0 0 ${chassis_z_offset + lidar_height}" rpy="0 0 0" />
 	</xacro:VLP-16>
 	<!-- IMU -->
@@ -107,20 +149,29 @@
 			</geometry>
 		</visual>
+        <collision name="imu_collision">
+            <origin xyz="0 0 0" rpy="0 0 0" />
+            <geometry>
+                <box size="${imu_length} ${imu_width} ${imu_height}" />
+            </geometry>
+        </collision>
+        <xacro:box_inertia mass="${imu_mass}" length="${imu_length}" width="${imu_width}" height="${imu_height}">
+            <origin xyz="0 0 0" rpy="0 0 0" />
+        </xacro:box_inertia>
 	</link>
 	<joint name="imu_joint" type="fixed">
-		<origin xyz="0 0 ${chassis_height/2}" rpy="0 0 0" />
+		<origin xyz="${-chassis_tower_length / 2 - chassis_electrical_length/2+0.005} 0 ${chassis_electrical_height + chassis_z_offset}" rpy="0 0 0" />
 		<parent link="chassis" />
 		<child link="imu_link" />
 		<axis xyz="0 1 0" />
 	</joint>
-	<!-- Encoders -->
-	<link name="encoders" />
+    <!-- Encoders -->
+    <link name="encoders" />
 	<joint name="encoders_joint" type="fixed">
-		<origin xyz="${front_offset} 0 ${wheel_offset-chassis_height/2}" rpy="0 0 0" />
+		<origin xyz="0 0 ${wheel_radius}" rpy="0 0 0" />
 		<parent link="chassis" />
 		<child link="encoders" />
 		<axis xyz="0 1 0" />
 	</joint>
-	<!-- Odom -->
+    <!-- Odom -->
 	<link name="odom" />
 	<joint name="odom_joint" type="fixed">
@@ -130,15 +181,15 @@
 		<axis xyz="0 1 0" />
 	</joint>
-	<!-- Color of bot -->
-	<gazebo reference="chassis_base_visual">
-		<material>Gazebo/Blue</material>
-	</gazebo>
-	<gazebo reference="chassis_top_visual">
-		<material>Gazebo/Blue</material>
-	</gazebo>
-	<gazebo reference="chassis_front_visual">
-		<material>Gazebo/Blue</material>
-	</gazebo>
-	<gazebo reference="chassis_back_visual">
+    <!-- Color of bot -->
+	<gazebo reference="chassis_tower_visual">
+		<material>Gazebo/Blue</material>
+	</gazebo>
+	<gazebo reference="chassis_payload_visual">
+		<material>Gazebo/Blue</material>
+	</gazebo>
+	<gazebo reference="chassis_electrical_visual">
+		<material>Gazebo/Blue</material>
+	</gazebo>
+	<gazebo reference="chassis_caster_visual">
 		<material>Gazebo/Blue</material>
 	</gazebo>
@@ -146,8 +197,8 @@
 		<material>Gazebo/Green</material>
 	</gazebo>
-	<gazebo reference="imu">
+	<gazebo reference="imu_visual">
 		<material>Gazebo/Purple</material>
 	</gazebo>
-	<!-- Motor, Camera and IMU Simulation -->
+    <!-- Motor, Camera and IMU Simulation -->
 	<xacro:include filename="$(find marvin_simulation)/urdf/marvin.gazebo" />
 </robot>

Commit message: Remove odom link for proper wheel transform

File: simulation/marvin_simulation/urdf/marvin.xacro (robot description, xacro)
@@ -173,12 +173,4 @@
 		<axis xyz="0 1 0" />
 	</joint>
-    <!-- Odom -->
-	<link name="odom" />
-	<joint name="odom_joint" type="fixed">
-		<origin xyz="0 0 0" rpy="0 0 0" />
-		<parent link="odom" />
-		<child link="chassis" />
-		<axis xyz="0 1 0" />
-	</joint>
     <!-- Color of bot -->
 	<gazebo reference="chassis_tower_visual">

Commit message: Move cog backwards by 4 inches to prevent tipping

File: simulation/marvin_simulation/urdf/marvin.xacro (robot description, xacro)
@@ -17,5 +17,5 @@
     <!-- Chassis Inertial Constants -->
     <xacro:property name="chassis_mass" value="29.9371" />
-    <xacro:property name="com_x" value="0.0" />
+    <xacro:property name="com_x" value="${-4.0*0.0254}" />
     <xacro:property name="com_y" value="0.0" />
     <xacro:property name="com_z" value="${6.1875*0.0254}" />

Commit message: Move base_link upwards and add base_footprint

File: simulation/marvin_simulation/urdf/marvin.xacro (robot description, xacro)
@@ -19,5 +19,5 @@
     <xacro:property name="com_x" value="${-4.0*0.0254}" />
     <xacro:property name="com_y" value="0.0" />
-    <xacro:property name="com_z" value="${6.1875*0.0254}" />
+    <xacro:property name="com_z" value="${6.1875*0.0254-chassis_z_offset}" />
 	<!-- Caster Constants -->
     <xacro:property name="caster_x_offset" value="${-24.625*0.0254}" />
@@ -45,5 +45,5 @@
 	<link name="base_link">
 		<visual name="chassis_tower_visual">
-			<origin xyz="0 0 ${chassis_tower_height / 2 + chassis_z_offset}" rpy="0 0 0" />
+			<origin xyz="0 0 ${chassis_tower_height / 2}" rpy="0 0 0" />
 			<geometry>
 				<box size="${chassis_tower_length} ${chassis_width} ${chassis_tower_height}" />
@@ -51,5 +51,5 @@
 		</visual>
         <visual name="chassis_payload_visual">
-            <origin xyz="${chassis_tower_length / 2 + chassis_payload_length / 2} 0 ${chassis_payload_height / 2 + chassis_z_offset}" rpy="0 0 0" />
+            <origin xyz="${chassis_tower_length / 2 + chassis_payload_length / 2} 0 ${chassis_payload_height / 2}" rpy="0 0 0" />
             <geometry>
                 <box size="${chassis_payload_length} ${chassis_width} ${chassis_payload_height}" />
@@ -57,5 +57,5 @@
         </visual>
         <visual name="chassis_electrical_visual">
-            <origin xyz="${-chassis_tower_length / 2 - chassis_electrical_length / 2} 0 ${chassis_electrical_height / 2 + chassis_z_offset}" rpy="0 0 0" />
+            <origin xyz="${-chassis_tower_length / 2 - chassis_electrical_length / 2} 0 ${chassis_electrical_height / 2}" rpy="0 0 0" />
             <geometry>
                 <box size="${chassis_electrical_length} ${chassis_width} ${chassis_electrical_height}" />
@@ -65,5 +65,5 @@
             <origin xyz="${-chassis_tower_length / 2 - chassis_electrical_length - chassis_caster_length / 2}
                          0
-                         ${chassis_caster_height / 2 + chassis_caster_z_offset + chassis_z_offset}"
+                         ${chassis_caster_height / 2 + chassis_caster_z_offset}"
                          rpy="0 0 0" />
             <geometry>
@@ -74,5 +74,5 @@
 			<origin xyz="${chassis_tower_length / 2 + chassis_payload_length - chassis_length / 2}
                          0
-                         ${chassis_z_offset + chassis_tower_height / 2}"
+                         ${chassis_tower_height / 2}"
                     rpy="0 0 0" />
 			<geometry>
@@ -84,4 +84,14 @@
 		</xacro:box_inertia>
 	</link>
+    <link name="base_footprint">
+        <xacro:box_inertia mass="0" length="0" width="0" height="0">
+            <origin xyz="0 0 0" rpy="0 0 0" />
+        </xacro:box_inertia>
+    </link>
+    <joint name="base_joint" type="fixed">
+        <origin xyz="0 0 ${-chassis_z_offset}" rpy="0 0 0" />
+        <parent link="base_link" />
+        <child link="base_footprint" />
+    </joint>
     <!-- Caster -->
     <link name="caster">
@@ -110,5 +120,5 @@
     </link>
     <joint name="caster_joint" type="fixed">
-        <origin xyz="${caster_x_offset} 0 ${caster_radius}" rpy="0 0 0" />
+        <origin xyz="${caster_x_offset} 0 ${caster_radius-chassis_z_offset}" rpy="0 0 0" />
         <parent link="base_link" />
         <child link="caster" />
@@ -117,8 +127,8 @@
     <xacro:include filename="$(find marvin_simulation)/urdf/wheel.xacro"/>
 	<xacro:wheel prefix="right" mass="${wheel_mass}" radius="${wheel_radius}" width="${wheel_width}">
-		<origin xyz="0 -${track_width / 2} ${wheel_radius}" rpy="0 0 0" />
+		<origin xyz="0 -${track_width / 2} ${wheel_radius-chassis_z_offset}" rpy="0 0 0" />
 	</xacro:wheel>
 	<xacro:wheel prefix="left" mass="${wheel_mass}" radius="${wheel_radius}" width="${wheel_width}">
-		<origin xyz="0 ${track_width/2} ${wheel_radius}" rpy="0 0 0" />
+		<origin xyz="0 ${track_width/2} ${wheel_radius-chassis_z_offset}" rpy="0 0 0" />
 	</xacro:wheel>
     <!-- ZED Camera -->
@@ -127,5 +137,5 @@
 	</xacro:zed_camera>
 	<joint name="zed_camera_joint" type="fixed">
-		<origin xyz="${camera_x_offset} 0 ${camera_z_offset + chassis_z_offset}" rpy="0 ${camera_angle} 0" />
+		<origin xyz="${camera_x_offset} 0 ${camera_z_offset}" rpy="0 ${camera_angle} 0" />
 		<parent link="base_link" />
 		<child link="zed_camera_link" />
@@ -134,10 +144,10 @@
 	<xacro:include filename="$(find marvin_simulation)/urdf/camera.xacro" />
 	<xacro:camera mass="${camera_mass}">
-		<origin xyz="${camera_x_offset} 0 ${camera_z_offset + chassis_z_offset}" rpy="0 ${camera_angle} 0" />
+		<origin xyz="${camera_x_offset} 0 ${camera_z_offset}" rpy="0 ${camera_angle} 0" />
 	</xacro:camera>
     <!-- Lidar -->
     <xacro:include filename="$(find velodyne_description)/urdf/VLP-16.urdf.xacro" />
 	<xacro:VLP-16 parent="base_link" name="velodyne" topic="/velodyne_points" hz="20" samples="440" gpu="true">
-		<origin xyz="0 0 ${chassis_z_offset + lidar_height}" rpy="0 0 0" />
+		<origin xyz="0 0 ${lidar_height}" rpy="0 0 0" />
 	</xacro:VLP-16>
 	<!-- IMU -->
@@ -160,5 +170,5 @@
 	</link>
 	<joint name="imu_joint" type="fixed">
-		<origin xyz="${-chassis_tower_length / 2 - chassis_electrical_length/2+0.005} 0 ${chassis_electrical_height + chassis_z_offset}" rpy="0 0 0" />
+		<origin xyz="${-chassis_tower_length / 2 - chassis_electrical_length/2+0.005} 0 ${chassis_electrical_height}" rpy="0 0 0" />
 		<parent link="base_link" />
 		<child link="imu_link" />
