Commit message: Final renaming

File: robot_description/marvin_description/urdf/constants.xacro (robot description, xacro)
@@ -30,12 +30,13 @@
     <xacro:property name="caster_mass" value="0.1" />
     <!-- Camera Mount Constants -->
-    <xacro:property name="camera_angle" value="${10 * 0.01745327777}"/>
     <xacro:property name="camera_x_offset" value="${chassis_tower_length/2 + 2.66916*0.0254}"/>
+    <xacro:property name="camera_y_offset" value="0.0"/>
     <xacro:property name="camera_z_offset" value="${chassis_z_offset + chassis_tower_height - 1.80395*0.0254}"/>
+    <xacro:property name="camera_pitch_offset" value="${10 * 0.01745327777}"/>
     <!-- IMU Constants -->
     <xacro:property name="imu_x_offset" value="0.0"/>
     <xacro:property name="imu_y_offset" value="0.0"/>
     <xacro:property name="imu_z_offset" value="${chassis_z_offset + chassis_tower_height}"/>
-    <xacro:property name="imu_yaw" value="${-pi/2}"/>
+    <xacro:property name="imu_yaw_offset" value="${-pi/2}"/>
     <!-- GPS Constants -->
     <xacro:property name="gps_x_offset" value="${3*0.0254}"/>

File: robot_description/marvin_description/urdf/marvin.xacro (robot description, xacro)
@@ -28,10 +28,10 @@
     <xacro:include filename="$(find common_description)/urdf/sensor/zed2i.xacro" />
     <xacro:zed2i name="$(arg zed_name)" parent="$(arg base_frame_id)">
-        <origin xyz="${camera_x_offset} 0 ${camera_z_offset}" rpy="0 ${camera_angle} 0" />
+        <origin xyz="${camera_x_offset} ${camera_y_offset} ${camera_z_offset}" rpy="0 ${camera_pitch_offset} 0" />
     </xacro:zed2i>
     <!-- IMU -->
     <xacro:include filename="$(find common_description)/urdf/sensor/vn300.xacro" />
     <xacro:vn300 name="$(arg imu_name)" parent="$(arg base_frame_id)">
-        <origin xyz="${imu_x_offset} ${imu_y_offset} ${imu_z_offset}" rpy="0 0 ${imu_yaw}" />
+        <origin xyz="${imu_x_offset} ${imu_y_offset} ${imu_z_offset}" rpy="0 0 ${imu_yaw_offset}" />
     </xacro:vn300>
     <!-- GPS -->
